File: Sistem Mikrokontroller/3. Membangun Sistem Minimum/Skematik1.sch (EAGLE design)
At the start: 19 parts, among them IC2 78L05Z, J1 DCJ0202, U1 328P

Commit message: update
Parts:
- removed C4: (no value), rcl:C-EU025-025X050
- removed S1: (no value), switch-omron:10-XX
- added JP4, JP5: (no value), pinhead:PINHD-1X10
- added S2: (no value), switch-omron:31-XX
Connections:
- removed net N$17: D1.A
- removed net N$18: SV1.2
- removed net N$19: U1.GND
- removed net N$20: U1.AVCC, U1.VCC
- new net N$21: D1.A, J1.1
- net GND: now also J1.2, J1.3, JP5.1, JP5.10, JP5.2, JP5.3, JP5.4, JP5.5, JP5.6, JP5.7, JP5.8, JP5.9, SV1.10, SV1.4, SV1.6, SV1.8, U1.GND
- net N$28: now also SV1.1
- net N$29: now also SV1.9
- net N$30: now also SV1.7
- net N$34: now also S2.P, SV1.5; no longer S1.P
- net N$37: now also C7.-, S2.S; no longer C4.2, S1.S
- net VCC: now also C7.+, JP4.1, JP4.10, JP4.2, JP4.3, JP4.4, JP4.5, JP4.6, JP4.7, JP4.8, JP4.9, SV1.2, U1.AVCC, U1.VCC; no longer C4.1
Other:
- moved on the sheet: C6, C7, J1, SV1

Commit message: update
Connections:
- removed net N$37: C3.2, C7.-, S2.S
- net GND: now also C3.2, C7.-, S2.S
Changed lines of the file:
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@@
 <part name="P+4" library="supply1" library_urn="urn:adsk.eagle:library:371" deviceset="VCC" device=""/>
 <part name="GND5" library="supply1" library_urn="urn:adsk.eagle:library:371" deviceset="GND" device=""/>
+<part name="GND6" library="supply1" library_urn="urn:adsk.eagle:library:371" deviceset="GND" device=""/>
 </parts>
 <sheets>
@@
 <instance part="GND5" gate="1" x="142.24" y="40.64" smashed="yes">
 <attribute name="VALUE" x="139.7" y="38.1" size="1.778" layer="96"/>
+</instance>
+<instance part="GND6" gate="1" x="78.74" y="91.44" smashed="yes">
+<attribute name="VALUE" x="76.2" y="88.9" size="1.778" layer="96"/>
 </instance>
 </instances>
@@
 <junction x="142.24" y="68.58"/>
 </segment>
+<segment>
+<wire x1="63.5" y1="104.14" x2="66.04" y2="104.14" width="0.1524" layer="91"/>
+<wire x1="66.04" y1="104.14" x2="66.04" y2="93.98" width="0.1524" layer="91"/>
+<pinref part="C3" gate="G$1" pin="2"/>
+<wire x1="66.04" y1="93.98" x2="60.96" y2="93.98" width="0.1524" layer="91"/>
+<wire x1="66.04" y1="93.98" x2="73.66" y2="93.98" width="0.1524" layer="91"/>
+<wire x1="73.66" y1="93.98" x2="73.66" y2="106.68" width="0.1524" layer="91"/>
+<junction x="66.04" y="93.98"/>
+<pinref part="C7" gate="G$1" pin="-"/>
+<pinref part="S2" gate="1" pin="S"/>
+<pinref part="GND6" gate="1" pin="GND"/>
+<wire x1="78.74" y1="93.98" x2="73.66" y2="93.98" width="0.1524" layer="91"/>
+<junction x="73.66" y="93.98"/>
+</segment>
 </net>
 <net name="N$34" class="0">
@@
 </segment>
 </net>
-<net name="N$37" class="0">
-<segment>
-<wire x1="63.5" y1="104.14" x2="66.04" y2="104.14" width="0.1524" layer="91"/>
-<wire x1="66.04" y1="104.14" x2="66.04" y2="93.98" width="0.1524" layer="91"/>
-<pinref part="C3" gate="G$1" pin="2"/>
-<wire x1="66.04" y1="93.98" x2="60.96" y2="93.98" width="0.1524" layer="91"/>
-<wire x1="66.04" y1="93.98" x2="73.66" y2="93.98" width="0.1524" layer="91"/>
-<wire x1="73.66" y1="93.98" x2="73.66" y2="106.68" width="0.1524" layer="91"/>
-<junction x="66.04" y="93.98"/>
-<pinref part="C7" gate="G$1" pin="-"/>
-<pinref part="S2" gate="1" pin="S"/>
-</segment>
-</net>
